File: kicad/main/main.kicad_sch (KiCad schematic)
At the start: 50 parts, among them J1 Conn_01x02, J10 Conn_01x02, J2 Conn_01x03, J3 Conn_01x03, J4 Conn_01x02, J5 Conn_01x02, J6 Connector, USB-TYPE-C-16P, J7 Conn_01x02, J8 Conn_01x02, U2 XC6206P332MR, U5 RP2040, X1 X322512MSB4SI

Commit message: Prorgess on PCB
Parts:
- added JP1: SolderJumper_2_Open, Jumper:SolderJumper-2_P1.3mm_Open_Pad1.0x1.5mm, symbol Jumper:SolderJumper_2_Open
Connections:
- net GND: now also JP1.1 (A)
- net at R10.1, R9.2: now also JP1.2 (B)
Other:
- moved on the sheet: R10
Changed lines of the file:
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@@
 	)
 	(junction
+		(at 224.79 69.85)
+		(diameter 0)
+		(color 0 0 0 0)
+	)
+	(junction
 		(at 96.52 27.94)
 		(diameter 0)
@@
 	)
 	(junction
+		(at 224.79 80.01)
+		(diameter 0)
+		(color 0 0 0 0)
+	)
+	(junction
 		(at 29.21 181.61)
 		(diameter 0)
@@
 	(wire
 		(pts
+			(xy 224.79 81.28) (xy 224.79 80.01)
+		)
+		(stroke
+			(width 0)
+			(type default)
+		)
+	)
+	(wire
+		(pts
 			(xy 81.28 182.88) (xy 82.55 182.88)
 		)
@@
 	(wire
 		(pts
+			(xy 224.79 69.85) (xy 224.79 68.58)
+		)
+		(stroke
+			(width 0)
+			(type default)
+		)
+	)
+	(wire
+		(pts
 			(xy 215.9 66.04) (xy 218.44 66.04)
 		)
@@
 	(wire
 		(pts
+			(xy 224.79 80.01) (xy 237.49 80.01)
+		)
+		(stroke
+			(width 0)
+			(type default)
+		)
+	)
+	(wire
+		(pts
 			(xy 29.21 167.64) (xy 29.21 181.61)
 		)
@@
 	(wire
 		(pts
+			(xy 224.79 69.85) (xy 237.49 69.85)
+		)
+		(stroke
+			(width 0)
+			(type default)
+		)
+	)
+	(wire
+		(pts
 			(xy 140.97 27.94) (xy 149.86 27.94)
 		)
@@
 	(wire
 		(pts
+			(xy 224.79 71.12) (xy 224.79 69.85)
+		)
+		(stroke
+			(width 0)
+			(type default)
+		)
+	)
+	(wire
+		(pts
 			(xy 72.39 33.02) (xy 72.39 30.48)
 		)
@@
 	(wire
 		(pts
+			(xy 224.79 80.01) (xy 224.79 78.74)
+		)
+		(stroke
+			(width 0)
+			(type default)
+		)
+	)
+	(wire
+		(pts
 			(xy 27.94 173.99) (xy 30.48 173.99)
 		)
@@
 	(symbol
 		(lib_id "PCM_JLCPCB-Resistors:1206,100mΩ")
-		(at 224.79 72.39 0)
+		(at 224.79 74.93 0)
 		(unit 1)
 		(body_style 1)
@@
 		(fields_autoplaced yes)
 		(property "Reference" "R10"
-			(at 227.33 72.3899 0)
+			(at 227.33 74.9299 0)
 			(show_name no)
 			(do_not_autoplace no)
@@
 		)
 		(property "Value" "100mΩ"
-			(at 224.79 72.39 90)
+			(at 224.79 74.93 90)
 			(show_name no)
 			(do_not_autoplace yes)
@@
 		)
 		(property "Footprint" "PCM_JLCPCB:R_1206"
-			(at 223.012 72.39 90)
+			(at 223.012 74.93 90)
 			(hide yes)
 			(show_name no)
@@
 		)
 		(property "Datasheet" "https://www.lcsc.com/datasheet/lcsc_datasheet_2205311900_UNI-ROYAL-Uniroyal-Elec-1206W4F100LT5E_C25334.pdf"
-			(at 224.79 72.39 0)
+			(at 224.79 74.93 0)
 			(hide yes)
 			(show_name no)
@@
 		)
 		(property "Description" "250mW Thick Film Resistors 200V ±800ppm/°C ±1% 100mΩ 1206 Chip Resistor - Surface Mount ROHS"
-			(at 224.79 72.39 0)
+			(at 224.79 74.93 0)
 			(hide yes)
 			(show_name no)
@@
 		)
 		(property "LCSC" "C25334"
-			(at 224.79 72.39 0)
+			(at 224.79 74.93 0)
 			(hide yes)
 			(show_name no)
@@
 		)
 		(property "Stock" "221617"
-			(at 224.79 72.39 0)
+			(at 224.79 74.93 0)
 			(hide yes)
 			(show_name no)
@@
 		)
 		(property "Price" "0.008USD"
-			(at 224.79 72.39 0)
+			(at 224.79 74.93 0)
 			(hide yes)
 			(show_name no)
@@
 		)
 		(property "Process" "SMT"
-			(at 224.79 72.39 0)
+			(at 224.79 74.93 0)
 			(hide yes)
 			(show_name no)
@@
 		)
 		(property "Minimum Qty" "15"
-			(at 224.79 72.39 0)
+			(at 224.79 74.93 0)
 			(hide yes)
 			(show_name no)
@@
 		)
 		(property "Attrition Qty" "10"
-			(at 224.79 72.39 0)
+			(at 224.79 74.93 0)
 			(hide yes)
 			(show_name no)
@@
 		)
 		(property "Class" "Basic Component"
-			(at 224.79 72.39 0)
+			(at 224.79 74.93 0)
 			(hide yes)
 			(show_name no)
@@
 		)
 		(property "Category" "Resistors,Chip Resistor - Surface Mount"
-			(at 224.79 72.39 0)
+			(at 224.79 74.93 0)
 			(hide yes)
 			(show_name no)
@@
 		)
 		(property "Manufacturer" "UNI-ROYAL(Uniroyal Elec)"
-			(at 224.79 72.39 0)
+			(at 224.79 74.93 0)
 			(hide yes)
 			(show_name no)
@@
 		)
 		(property "Part" "1206W4F100LT5E"
-			(at 224.79 72.39 0)
+			(at 224.79 74.93 0)
 			(hide yes)
 			(show_name no)
@@
 		)
 		(property "Resistance" "100mΩ"
-			(at 224.79 72.39 0)
+			(at 224.79 74.93 0)
 			(hide yes)
 			(show_name no)
@@
 		)
 		(property "Power(Watts)" "250mW"
-			(at 224.79 72.39 0)
+			(at 224.79 74.93 0)
 			(hide yes)
 			(show_name no)
@@
 		)
 		(property "Type" "Thick Film Resistors"
-			(at 224.79 72.39 0)
+			(at 224.79 74.93 0)
 			(hide yes)
 			(show_name no)
@@
 		)
 		(property "Overload Voltage (Max)" "200V"
-			(at 224.79 72.39 0)
+			(at 224.79 74.93 0)
 			(hide yes)
 			(show_name no)
@@
 		)
 		(property "Operating Temperature Range" "-55°C~+155°C"
-			(at 224.79 72.39 0)
+			(at 224.79 74.93 0)
 			(hide yes)
 			(show_name no)
@@
 		)
 		(property "Tolerance" "±1%"
-			(at 224.79 72.39 0)
+			(at 224.79 74.93 0)
 			(hide yes)
 			(show_name no)
@@
 		)
 		(property "Temperature Coefficient" "±800ppm/°C"
-			(at 224.79 72.39 0)
+			(at 224.79 74.93 0)
 			(hide yes)
 			(show_name no)
@@
 	(symbol
 		(lib_id "power:GND")
-		(at 224.79 76.2 0)
+		(at 224.79 81.28 0)
 		(unit 1)
 		(body_style 1)
@@
 		(fields_autoplaced yes)
 		(property "Reference" "#PWR039"
-			(at 224.79 82.55 0)
+			(at 224.79 87.63 0)
 			(hide yes)
 			(show_name no)
@@
 		)
 		(property "Value" "GND"
-			(at 224.79 81.28 0)
+			(at 224.79 86.36 0)
 			(show_name no)
 			(do_not_autoplace no)
@@
 		)
 		(property "Footprint" ""
-			(at 224.79 76.2 0)
+			(at 224.79 81.28 0)
 			(hide yes)
 			(show_name no)
@@
 		)
 		(property "Datasheet" ""
-			(at 224.79 76.2 0)
+			(at 224.79 81.28 0)
 			(hide yes)
 			(show_name no)
@@
 		)
 		(property "Description" "Power symbol creates a global label with name \"GND\" , ground"
-			(at 224.79 76.2 0)
+			(at 224.79 81.28 0)
 			(hide yes)
 			(show_name no)
@@
 					(unit 1)
 				)
+			)
+		)
+	)
+	(symbol
+		(lib_id "Jumper:SolderJumper_2_Open")
+		(at 237.49 74.93 90)
+		(unit 1)
+		(body_style 1)
+		(exclude_from_sim no)
+		(in_bom no)
+		(on_board yes)
+		(in_pos_files yes)
+		(dnp no)
+		(fields_autoplaced yes)
+		(property "Reference" "JP1"
+			(at 240.03 73.6599 90)
+			(show_name no)
+			(do_not_autoplace no)
+			(effects
+				(font
+					(size 1.27 1.27)
+				)
+				(justify right)
+			)
+		)
+		(property "Value" "SolderJumper_2_Open"
+			(at 240.03 76.1999 90)
+			(hide yes)
+			(show_name no)
+			(do_not_autoplace no)
+			(effects
+				(font
+					(size 1.27 1.27)
+				)
+				(justify right)
+			)
+		)
+		(property "Footprint" "Jumper:SolderJumper-2_P1.3mm_Open_Pad1.0x1.5mm"
+			(at 237.49 74.93 0)
+			(hide yes)
+			(show_name no)
+			(do_not_autoplace no)
+			(effects
+				(font
+					(size 1.27 1.27)
+				)
+			)
+		)
+		(property "Datasheet" ""
+			(at 245.11 74.93 0)
+			(hide yes)
+			(show_name no)
+			(do_not_autoplace no)
+			(effects
+				(font
+					(size 1.27 1.27)
+				)
+			)
+		)
+		(property "Description" "Solder Jumper, 2-pole, open"
+			(at 242.57 74.93 0)
+			(hide yes)
+			(show_name no)
+			(do_not_autoplace no)
+			(effects
+				(font
+					(size 1.27 1.27)
+				)
+			)
+		)
+		(pin "1"
+		)
+		(pin "2"
+		)
+		(instances
+			(project "main"
+				(path "/04d416a6-c3f6-4cc1-b329-31df85c27013"
+					(reference "JP1")
+					(unit 1)
+				)

Commit message: Progress on PCB design
Parts:
- added H1, H2: MountingHole, MountingHole:MountingHole_2.5mm, symbol Mechanical:MountingHole
- added R1, R11: 10kΩ, PCM_JLCPCB:R_0402, symbol PCM_JLCPCB-Resistors:0402,10kΩ
Connections:
- net GND: now also R1.2, R11.2
- net T Board: now also R1.1
- net T LED: now also R11.1
Other:
- moved on the sheet: J1, J4, J5
