File: kicad/main/main.kicad_pcb (KiCad board)
At the start: 2 copper layers, 32.4 x 26.8 mm, 52 parts, among them J1 Conn_01x02, J10 Conn_01x02, J2 Conn_01x03, J3 Conn_01x03, J4 Conn_01x02, J5 Conn_01x02, J6 Connector, USB-TYPE-C-16P, J7 Conn_01x02, J8 Conn_01x02, U2 XC6206P332MR, U5 RP2040, X1 X322512MSB4SI

Commit message: Progress on fixing issues
Parts:
- removed R8: 430Ω, PCM_JLCPCB:R_0603
- added C17: 10uF, PCM_JLCPCB:C_0805, F.Cu at (106.4, 53.4)
- added C18: 10uF, PCM_JLCPCB:C_0805, F.Cu at (121.2, 39.0)
- added D1: SS34, PCM_JLCPCB:D_SMA, F.Cu at (128.2, 49.6)
- moved J7 5.10 mm to (120.3, 53.7)
- moved J8 5.10 mm to (125.4, 53.7)
- moved TP4 2.00 mm to (116.5, 53.0)
- moved TP3 1.82 mm to (115.0, 54.4)
- moved TP2 1.70 mm to (113.0, 53.9)
Connections:
- J2 pad 1: +5V -> Pan
- J2 pad 2: Pan -> +5V
- J3 pad 1: +5V -> Tilt
- J3 pad 2: Tilt -> +5V
- J7 pad 1: +5V -> Net-(J7-Pin_1)
- J8 pad 1: +5V -> Net-(J7-Pin_1)
Routing:
- net GND: track 69.1 -> 89.4 mm
- net +5V: track 86.4 -> 94.2 mm, vias 2 -> 4
- net Net-(J7-Pin_1): track 0.00 -> 7.50 mm
- net Tilt: track 38.3 -> 35.8 mm
- net Net-(U5-GPIO6): track 4.50 -> 2.49 mm
- net Pan: track 28.2 -> 26.3 mm
- net Net-(U5-GPIO4): track 2.08 -> 3.55 mm
